Commit message: remove ground fixed joint

File: 3dof.urdf (robot description, URDF)
Before this commit: robot simple_3dof_arm, 4 links, 3 joints
Links:
- added link payload, mass 1.0; collision sphere radius=0.05; visual sphere radius=0.05
Joints:
- added joint link3_to_payload: type fixed, parent link3, child payload, origin xyz=0.3 0 0 rpy=0 0 0

Commit message: A bit better

File: 3dof.urdf (robot description, URDF)
Before this commit: robot simple_3dof_arm, 5 links, 4 joints
Links:
- link link1: geometry collision box size=0.05 0.05 1; visual box size=0.05 0.05 1
Joints:
- joint joint1: origin xyz=0 0 0.5 rpy=0 0 0 -> xyz=0 0 1 rpy=0 0 0

Commit message: WIP

File: 3dof.urdf (robot description, URDF)
Before this commit: robot simple_3dof_arm, 5 links, 4 joints
Links:
- link link1: geometry collision box size=0.05 0.05 0.5; visual box size=0.05 0.05 0.5
Joints:
- joint joint1: origin xyz=0 0 1 rpy=0 0 0 -> xyz=0 0 0.5 rpy=0 0 0

Commit message: Graph mean torque and acc, modify base

File: 3dof.urdf (robot description, URDF)
Before this commit: robot simple_3dof_arm, 5 links, 4 joints
Links:
- added link motor_transmission_0, mass 0.9; collision box size=0.1 0.06 0.06; visual box size=0.1 0.06 0.06
- added link motor_transmission_1, mass 0.9; collision box size=0.1 0.06 0.06; visual box size=0.1 0.06 0.06
- added link motor_transmission_2, mass 0.9; collision box size=0.1 0.06 0.06; visual box size=0.1 0.06 0.06
- link ground_link: mass 5.0 -> 20.0; geometry collision box size=0.4 0.4 1.0; visual box size=0.4 0.4 1.0
Joints:
- added joint joint0_motor_transmission: type fixed, parent ground_link, child motor_transmission_0, origin xyz=0 0 0 rpy=0 0 0
- added joint joint1_motor_transmission: type fixed, parent link1, child motor_transmission_1, origin xyz=0 0 1 rpy=0 0 0
- added joint joint2_motor_transmission: type fixed, parent link2, child motor_transmission_2, origin xyz=0.3 0 0 rpy=0 0 0

Commit message: More like bot

File: 3dof.urdf (robot description, URDF)
Before this commit: robot simple_3dof_arm, 8 links, 7 joints
Links:
- link link1: geometry collision cylinder length=0.05 radius=0.1; visual cylinder length=0.05 radius=0.1
- link link2: mass 1.0 -> 2.0; geometry collision box size=0.8 0.05 0.05; visual box size=0.8 0.05 0.05
- link link3: mass 0.8 -> 2.0; geometry collision box size=0.8 0.05 0.05; visual box size=0.8 0.05 0.05
Joints:
- joint joint0: origin xyz=0 0 0 rpy=0 0 0 -> xyz=0 0 1.0 rpy=0 0 0
- joint joint0_motor_transmission: origin xyz=0 0 0 rpy=0 0 0 -> xyz=0 0 1.0 rpy=0 0 0
- joint joint1: origin xyz=0 0 1 rpy=0 0 0 -> xyz=0 0 0.05 rpy=0 0 0
- joint joint1_motor_transmission: origin xyz=0 0 1 rpy=0 0 0 -> xyz=0 0 0.05 rpy=0 0 0
- joint joint2: origin xyz=0.3 0 0 rpy=0 0 0 -> xyz=0.8 0 0 rpy=0 0 0
- joint joint2_motor_transmission: origin xyz=0.3 0 0 rpy=0 0 0 -> xyz=0.8 0 0 rpy=0 0 0
- joint link3_to_payload: origin xyz=0.3 0 0 rpy=0 0 0 -> xyz=0.8 0 0 rpy=0 0 0
